Commit message: Added hint managing

File: urdf/robot.urdf (robot description, URDF)
Before this commit: robot robot_xacro, 7 links, 6 joints
Links:
- link arm_link_01: geometry collision cylinder length=0.8 radius=0.04; visual cylinder length=0.7 radius=0.04
Joints:
- joint camera_joint: origin xyz=0.05 0 0.7 rpy=0 0 0 -> xyz=0.05 0 0.7 rpy=0 0.436332 0

Commit message: Adjusted movement

File: urdf/robot.urdf (robot description, URDF)
Before this commit: robot robot_xacro, 7 links, 6 joints
Links:
- added link camera2_link, mass 1e-5; collision box size=0.05 0.05 0.05; visual box size=0.05 0.05 0.05
Joints:
- added joint camera2_joint: type fixed, parent link_chassis, child camera2_link, origin xyz=0.25 0 0.01 rpy=0 0 0, axis 0 1 0
